File: circuit/circuit.kicad_sch (KiCad schematic)
At the start: 1 part, among them U1 Pico

Commit message: .
Parts:
- added D1, D2: 1N4148, Diode_THT:D_DO-35_SOD27_P7.62mm_Horizontal, symbol Diode:1N4148
- added J1: Micro_SD_Card, symbol Connector:Micro_SD_Card
- added J2: VGA, symbol Connector:DE15_Receptacle_HighDensity
- added J3: USB-C Power, symbol Connector:USB_C_Receptacle_PowerOnly_6P
- added J?: FTDI cable, symbol Connector_Generic:Conn_01x06
- added R1, R2, R3, R4, R5, R6, R7: 220, symbol Device:R
- added RV1: Trim 200, symbol Device:R_Potentiometer_Trim
- added U2: Z80CPU, symbol CPU:Z80CPU
- added U3: AS6C4008-55PCN, Package_DIP:DIP-32_W15.24mm, symbol Memory_RAM:AS6C4008-55PCN
- added U4, U5, U6: TXS0108EPW, Package_SO:TSSOP-20_4.4x6.5mm_P0.65mm, symbol Logic_LevelTranslator:TXS0108EPW
- added U7: 74LS393, symbol 74xx:74LS393
- added X1: 10Mhz, Oscillator:Oscillator_DIP-14, symbol Oscillator:CXO_DIP14
Connections:
- net at U1.1 (GPIO0): now also U4.20 (B1)
- net at U1.10 (GPIO7): now also U4.12 (B8)
- net at U1.11 (GPIO8): now also U5.20 (B1)
- net at U1.12 (GPIO9): now also U5.18 (B2)
- net at U1.14 (GPIO10): now also U5.17 (B3)
- net VSYNC: now reaches U1.15 (GPIO11)
- net VSYNC: now also J2.14
- net HSYNC: now reaches U1.16 (GPIO12)
- net HSYNC: now also J2.13, U5.16 (B4)
- net GREEN0: now reaches U1.17 (GPIO13)
- net GREEN0: now also R4.1, U5.15 (B5)
- net GREEN1: now reaches U1.19 (GPIO14)
- net GREEN1: now also R2.1, R5.2, R6.2, RV1.1
- net at U1.2 (GPIO1): now also U4.18 (B2)
- net RED: now reaches U1.20 (GPIO15)
- net RED: now also R1.1
- net BLUE: now reaches U1.21 (GPIO16)
- net BLUE: now also R3.1
- net at U1.22 (GPIO17): now also U5.14 (B6)
- net GND: now reaches U1.23 (GND)
- net GND: now also D1.1 (K), D2.1 (K), J1.6 (VSS), J2.10, J2.5, J2.6, J2.7, J2.8, J3.A12 (GND), J3.B12 (GND), J?.1 (Pin_1), R7.1, RV1.2, U4.11 (GND), U5.11 (GND), U6.11 (GND), X1.7 (GND)
- net SCK: now reaches U1.24 (GPIO18)
- net SCK: now also J1.5 (CLK)
- net MOSI: now reaches U1.25 (GPIO19)
- net MOSI: now also J1.3 (CMD)
- net MISO: now reaches U1.26 (GPIO20)
- net MISO: now also J1.7 (DAT0)
- net CS: now reaches U1.27 (GPIO21)
- net CS: now also J1.2 (DAT3/CD)
- net at U1.29 (GPIO22): now also U5.13 (B7)
- net at U1.31 (GPIO26_ADC0): now also U5.12 (B8)
- net at U1.32 (GPIO27_ADC1): now also U6.18 (B2)
- net at U1.34 (GPIO28_ADC2): now also U6.20 (B1)
- net +3.3V: now reaches U1.36 (3V3)
- net +3.3V: now also J1.4 (VDD), U4.19 (VCCB), U5.19 (VCCB), U6.19 (VCCB)
- net +5V: now reaches U1.39 (VSYS)
- net +5V: now also J3.A9 (VBUS), J3.B9 (VBUS), J?.3 (Pin_3), U2.11 (VCC), U2.16 (~{INT}), U2.17 (~{NMI}), U2.18 (~{HALT}), U2.25 (~{BUSRQ}), U4.10 (OE), U4.2 (VCCA), U5.10 (OE), U5.2 (VCCA), U6.10 (OE), U6.2 (VCCA), X1.1 (EN), X1.14 (Vcc)
- net at U1.4 (GPIO2): now also U4.17 (B3)
- net at U1.5 (GPIO3): now also U4.16 (B4)
- net at U1.6 (GPIO4): now also U4.15 (B5)
- net at U1.7 (GPIO5): now also U4.14 (B6)
- net at U1.9 (GPIO6): now also U4.13 (B7)
- new net: D1.2 (A), J2.1, R1.2
- new net: J2.2, R2.2
- new net: D2.2 (A), J2.3, R3.2
- new net: U2.6 (~{CLK}), X1.8 (OUT)
- new net: U3.2 (A16), U7.3 (Q0)
- new net: U3.30 (A17), U7.4 (Q1)
- new net: U3.1 (A18), U7.5 (Q2)
- new net: R4.2, R5.1, R6.1, R7.2
- new net: U2.32 (A2), U3.10 (A2)
- new net: U2.31 (A1), U3.11 (A1)
- new net: U2.30 (A0), U3.12 (A0)
- new net: U2.40 (A10), U3.23 (A10)
- new net: U2.1 (A11), U3.25 (A11)
- new net: U2.39 (A9), U3.26 (A9)
- new net: U2.38 (A8), U3.27 (A8)
- new net: U2.3 (A13), U3.28 (A13)
- new net: U2.4 (A14), U3.3 (A14)
- new net: U2.5 (A15), U3.31 (A15)
- new net: U2.2 (A12), U3.4 (A12)
- new net: U2.37 (A7), U3.5 (A7)
- new net: U2.36 (A6), U3.6 (A6)
- new net: U2.35 (A5), U3.7 (A5)
- new net: U2.34 (A4), U3.8 (A4)
- new net: U2.33 (A3), U3.9 (A3)
- new net A0: U4.1 (A1)
- new net A1: U4.3 (A2)
- new net A2: U4.4 (A3)
- new net BANK: U5.7 (A6), U7.1 (CP)
- new net CTS: J?.2 (Pin_2)
- new net D0: U2.14 (D0), U3.13 (DQ0), U4.5 (A4)
- new net D1: U2.15 (D1), U3.14 (DQ1), U4.6 (A5)
- new net D2: U2.12 (D2), U3.15 (DQ2), U4.7 (A6)
- new net D3: U2.8 (D3), U3.17 (DQ3), U4.8 (A7)
- new net D4: U2.7 (D4), U3.18 (DQ4), U4.9 (A8)
- new net D5: U2.9 (D5), U3.19 (DQ5), U5.1 (A1)
- new net D6: U2.10 (D6), U3.20 (DQ6), U5.3 (A2)
- new net D7: U2.13 (D7), U3.21 (DQ7), U5.4 (A3)
- new net DTR: J?.6 (Pin_6)
- new net PCRX: J?.5 (Pin_5), U5.5 (A4)
- new net PCTX: J?.4 (Pin_4), U5.6 (A5)
- new net RST: U7.2 (MR)
- new net ~{IRQ}: U2.20 (~{IORQ}), U5.9 (A8)
- new net ~{MREQ}: U2.19 (~{MREQ}), U3.22 (CE#)
- new net ~{RD}: U2.21 (~{RD}), U3.24 (OE#)
- new net ~{RST}: U2.26 (~{RESET}), U6.3 (A2)
- new net ~{WAIT}: U2.24 (~{WAIT}), U5.8 (A7)
- new net ~{WR}: U2.22 (~{WR}), U3.29 (WE#), U6.1 (A1)
- no-connect marks 0 -> 39
Other:
- note added: "TODO: - find a place for ~{MREQ} - reorganize VGA pins"
- moved on the sheet: U1

Commit message: .
Parts:
- removed D1, D2: 1N4148, Diode_THT:D_DO-35_SOD27_P7.62mm_Horizontal, symbol Diode:1N4148
- removed J1: Micro_SD_Card, symbol Connector:Micro_SD_Card
- removed J2: VGA, symbol Connector:DE15_Receptacle_HighDensity
- removed J3: USB-C Power, symbol Connector:USB_C_Receptacle_PowerOnly_6P
- removed J?: FTDI cable, symbol Connector_Generic:Conn_01x06
- removed R1, R2, R3, R4, R5, R6, R7: 220, symbol Device:R
- removed RV1: Trim 200, symbol Device:R_Potentiometer_Trim
- removed U1: Pico, RPi_Pico:RPi_Pico_SMD_TH, symbol MCU_RaspberryPi_and_Boards:Pico
- removed U2: Z80CPU, symbol CPU:Z80CPU
- removed U3: AS6C4008-55PCN, Package_DIP:DIP-32_W15.24mm, symbol Memory_RAM:AS6C4008-55PCN
- removed U4, U5, U6: TXS0108EPW, Package_SO:TSSOP-20_4.4x6.5mm_P0.65mm, symbol Logic_LevelTranslator:TXS0108EPW
- removed U7: 74LS393, symbol 74xx:74LS393
- removed X1: 10Mhz, Oscillator:Oscillator_DIP-14, symbol Oscillator:CXO_DIP14
Connections:
- no-connect marks 39 -> 0
Other:
- added sheet Computer (computer.kicad_sch)
- added sheet IO (io.kicad_sch)
- note removed: "TODO: - find a place for ~{MREQ} - reorganize VGA pins"
