File: circuit/computer.kicad_sch (KiCad schematic)
At the start: 14 parts, among them J1 Mega2560 Left, J3 USB-C Power, J4 Mega2560 Right, J5 Ext. Clock, J7 IO, SW2 Debug, U2 Z80CPU, U3 AS6C4008-55PCN

Commit message: .
Parts:
- removed J7: IO, symbol Connector_Generic:Conn_01x21
- added C?: 1uF, symbol Device:C
- added D?: 1N4148, Diode_THT:D_DO-35_SOD27_P7.62mm_Horizontal, symbol Diode:1N4148
- added J2: Conn_01x22, symbol Connector_Generic:Conn_01x22
- added R2, R3, R4, R5: 10k, symbol Device:R
- added R?: 1K, symbol Device:R_US
- added R?: 100, symbol Device:R_US
- added SW?: RESET, symbol Switch:SW_Push
Connections:
- net +5V: now also J2.1 (Pin_1), R2.1
- net A0: now also J2.2 (Pin_2)
- net A1: now also J2.3 (Pin_3)
- net A16: now also J2.17 (Pin_17), R5.1
- net A17: now also J2.18 (Pin_18), R4.1
- net A18: now also J2.19 (Pin_19), R3.1
- net A2: now also J2.4 (Pin_4)
- net CLKENA: no longer J4.24 (Pin_24)
- net D0: now also J2.5 (Pin_5)
- net D1: now also J2.6 (Pin_6)
- net D2: now also J2.7 (Pin_7)
- net D3: now also J2.8 (Pin_8)
- net D4: now also J2.9 (Pin_9)
- net D5: now also J2.10 (Pin_10)
- net D6: now also J2.11 (Pin_11)
- net D7: now also J2.12 (Pin_12)
- net GND: now also C?.2, J2.22 (Pin_22), R3.2, R4.2, R5.2, SW?.1
- net ~{CLK}: now also J4.26 (Pin_26); no longer J4.25 (Pin_25)
- net ~{IORQ}: now also J2.13 (Pin_13)
- net ~{MREQ}: now also J2.14 (Pin_14)
- net ~{RST}: now also J4.27 (Pin_27), C?.1, D?.2 (A), J2.20 (Pin_20), R2.2, R?.1, R?.1; no longer J4.26 (Pin_26)
- net ~{WAIT}: now also J2.16 (Pin_16)
- net ~{WR}: now also J2.15 (Pin_15)
- net ~{IO_CE}: now reaches J4.28 (Pin_28)
- net ~{IO_CE}: now also J2.21 (Pin_21)
- net ~{M1}: now reaches U2.27 (~{M1})
- net ~{M1}: now also J4.24 (Pin_24)
- new net: R?.2, SW?.2
- new net VCC: D?.1 (K), R?.2
- new net ~{CLKENA}: J4.25 (Pin_25)
- no-connect marks 4 -> 3
Other:
- note added: "CPU & MEMORY"
- note added: "DEBUGGER"
- note added: "I/O"
- note added: "POWER"
- note added: "RESET"
- note removed: "MEGA2560 debugger"

Commit message: .
Connections:
- net A0: now also J1.28 (Pin_28); no longer J1.29 (Pin_29)
- net A1: now also J1.29 (Pin_29); no longer J1.30 (Pin_30)
- net A10: now also J4.8 (Pin_8); no longer J4.7 (Pin_7)
- net A11: now also J4.6 (Pin_6); no longer J4.5 (Pin_5)
- net A12: now also J1.36 (Pin_36); no longer J1.7 (Pin_7)
- net A13: now also J4.3 (Pin_3); no longer J4.2 (Pin_2)
- net A14: now also J1.7 (Pin_7); no longer J1.8 (Pin_8)
- net A15: now also J4.32 (Pin_32); no longer J4.31 (Pin_31)
- net A16: now also J1.8 (Pin_8); no longer J1.9 (Pin_9)
- net A17: now also J4.1 (Pin_1); no longer J4.32 (Pin_32)
- net A18: now also J1.9 (Pin_9); no longer J1.10 (Pin_10)
- net A2: now also J1.30 (Pin_30); no longer J1.31 (Pin_31)
- net A3: now also J1.31 (Pin_31); no longer J1.32 (Pin_32)
- net A4: now also J1.32 (Pin_32); no longer J1.33 (Pin_33)
- net A5: now also J1.33 (Pin_33); no longer J1.34 (Pin_34)
- net A6: now also J1.34 (Pin_34); no longer J1.35 (Pin_35)
- net A7: now also J1.35 (Pin_35); no longer J1.36 (Pin_36)
- net A8: now also J4.4 (Pin_4); no longer J4.3 (Pin_3)
- net A9: now also J4.5 (Pin_5); no longer J4.4 (Pin_4)
- net D0: now also J1.27 (Pin_27); no longer J1.28 (Pin_28)
- net D1: now also J1.26 (Pin_26); no longer J1.27 (Pin_27)
- net D2: now also J1.25 (Pin_25); no longer J1.26 (Pin_26)
- net D3: now also J4.14 (Pin_14); no longer J4.13 (Pin_13)
- net D4: now also J4.13 (Pin_13); no longer J4.12 (Pin_12)
- net D5: now also J4.12 (Pin_12); no longer J4.11 (Pin_11)
- net D6: now also J4.11 (Pin_11); no longer J4.10 (Pin_10)
- net D7: now also J4.10 (Pin_10); no longer J4.9 (Pin_9)
- net ~{BUSACK}: now also J4.23 (Pin_23); no longer J4.20 (Pin_20)
- net ~{BUSRQ}: now also J4.24 (Pin_24); no longer J4.21 (Pin_21)
- net ~{CLKENA}: now also J4.28 (Pin_28); no longer J4.25 (Pin_25)
- net ~{CLK}: now also J4.29 (Pin_29); no longer J4.26 (Pin_26)
- net ~{IORQ}: now also J4.25 (Pin_25), J4.26 (Pin_26); no longer J4.22 (Pin_22), J4.23 (Pin_23)
- net ~{IO_CE}: now also J4.31 (Pin_31); no longer J4.28 (Pin_28)
- net ~{M1}: now also J4.27 (Pin_27); no longer J4.24 (Pin_24)
- net ~{MREQ}: now also J4.9 (Pin_9); no longer J4.8 (Pin_8)
- net ~{RD}: now also J4.7 (Pin_7); no longer J4.6 (Pin_6)
- net ~{RST}: now also J4.30 (Pin_30); no longer J4.27 (Pin_27)
- net ~{WR}: now also J4.2 (Pin_2); no longer J4.1 (Pin_1)
- net at SW2.1: now also J4.17 (Pin_17); no longer J4.30 (Pin_30)

Commit message: .
Connections:
- net +5V: no longer U2.17 (~{NMI})
- net ~{BUSACK}: now also J4.24 (Pin_24); no longer J4.23 (Pin_23)
- net ~{BUSRQ}: now also J4.25 (Pin_25); no longer J4.24 (Pin_24)
- net ~{IORQ}: no longer J4.25 (Pin_25)
- net ~{WAIT}: now also J4.22 (Pin_22)
- new net ~{NMI}: J4.23 (Pin_23), U2.17 (~{NMI})
Changed lines of the file:
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@@
   (junction (at 249.428 125.984) (diameter 0) (color 0 0 0 0)
   )
-  (junction (at 113.665 27.432) (diameter 0) (color 0 0 0 0)
-  )
-  (junction (at 113.665 50.292) (diameter 0) (color 0 0 0 0)
-  )
   (junction (at 133.35 27.432) (diameter 0) (color 0 0 0 0)
+  )
+  (junction (at 113.538 27.432) (diameter 0) (color 0 0 0 0)
   )
   (junction (at 105.664 35.052) (diameter 0) (color 0 0 0 0)
@@
     (stroke (width 0) (type default))
   )
-  (wire (pts (xy 113.665 50.292) (xy 113.665 27.432))
-    (stroke (width 0) (type default))
-  )
   (wire (pts (xy 37.338 80.772) (xy 46.99 80.772))
     (stroke (width 0) (type default))
@@
     (stroke (width 0) (type default))
   )
-  (wire (pts (xy 113.665 52.832) (xy 113.665 50.292))
-    (stroke (width 0) (type default))
-  )
   (wire (pts (xy 176.53 45.212) (xy 151.13 45.212))
     (stroke (width 0) (type default))
@@
     (stroke (width 0) (type default))
   )
+  (wire (pts (xy 113.538 27.432) (xy 113.538 52.832))
+    (stroke (width 0) (type default))
+  )
   (wire (pts (xy 37.338 83.312) (xy 46.99 83.312))
     (stroke (width 0) (type default))
@@
     (stroke (width 0) (type default))
   )
-  (wire (pts (xy 113.665 27.432) (xy 133.35 27.432))
+  (wire (pts (xy 105.664 27.432) (xy 113.538 27.432))
     (stroke (width 0) (type default))
   )
@@
     (stroke (width 0) (type default))
   )
-  (wire (pts (xy 115.57 50.292) (xy 113.665 50.292))
+  (wire (pts (xy 103.378 50.292) (xy 115.57 50.292))
     (stroke (width 0) (type default))
   )
@@
     (stroke (width 0) (type default))
   )
-  (wire (pts (xy 105.664 27.432) (xy 113.665 27.432))
-    (stroke (width 0) (type default))
-  )
   (wire (pts (xy 236.728 125.984) (xy 236.728 129.794))
     (stroke (width 0) (type default))
@@
     (stroke (width 0) (type default))
   )
+  (wire (pts (xy 113.538 27.432) (xy 133.35 27.432))
+    (stroke (width 0) (type default))
+  )
   (wire (pts (xy 163.195 37.592) (xy 151.13 37.592))
     (stroke (width 0) (type default))
@@
     (stroke (width 0) (type default))
   )
+  (wire (pts (xy 90.424 162.814) (xy 101.6 162.814))
+    (stroke (width 0) (type default))
+  )
   (wire (pts (xy 69.342 152.654) (xy 77.724 152.654))
     (stroke (width 0) (type default))
@@
     (stroke (width 0) (type default))
   )
-  (wire (pts (xy 115.57 52.832) (xy 113.665 52.832))
+  (wire (pts (xy 113.538 52.832) (xy 115.57 52.832))
     (stroke (width 0) (type default))
   )
@@
     (effects (font (size 1.27 1.27)) (justify right bottom))
   )
+  (label "~{BUSRQ}" (at 101.6 155.194 180) (fields_autoplaced)
+    (effects (font (size 1.27 1.27)) (justify right bottom))
+  )
   (label "A0" (at 60.452 160.02 180) (fields_autoplaced)
     (effects (font (size 1.27 1.27)) (justify right bottom))
@@
     (effects (font (size 1.27 1.27)) (justify left bottom))
   )
-  (label "~{IORQ}" (at 101.6 155.194 180) (fields_autoplaced)
-    (effects (font (size 1.27 1.27)) (justify right bottom))
-  )
   (label "D4" (at 213.995 45.212 180) (fields_autoplaced)
     (effects (font (size 1.27 1.27)) (justify right bottom))
@@
     (effects (font (size 1.27 1.27)) (justify right bottom))
   )
+  (label "~{BUSACK}" (at 101.6 157.734 180) (fields_autoplaced)
+    (effects (font (size 1.27 1.27)) (justify right bottom))
+  )
   (label "~{CLKENA}" (at 101.346 147.574 180) (fields_autoplaced)
     (effects (font (size 1.27 1.27)) (justify right bottom))
   )
+  (label "~{NMI}" (at 101.6 160.274 180) (fields_autoplaced)
+    (effects (font (size 1.27 1.27)) (justify right bottom))
+  )
   (label "A11" (at 69.342 150.114 0) (fields_autoplaced)
     (effects (font (size 1.27 1.27)) (justify left bottom))
@@
     (effects (font (size 1.27 1.27)) (justify right bottom))
   )
+  (label "~{WAIT}" (at 101.6 162.814 180) (fields_autoplaced)
+    (effects (font (size 1.27 1.27)) (justify right bottom))
+  )
   (label "~{WR}" (at 69.342 139.954 0) (fields_autoplaced)
     (effects (font (size 1.27 1.27)) (justify left bottom))
@@
     (effects (font (size 1.27 1.27)) (justify left bottom))
   )
-  (label "~{BUSRQ}" (at 101.6 157.734 180) (fields_autoplaced)
-    (effects (font (size 1.27 1.27)) (justify right bottom))
-  )
   (label "D6" (at 69.342 162.814 0) (fields_autoplaced)
     (effects (font (size 1.27 1.27)) (justify left bottom))
@@
     (effects (font (size 1.27 1.27)) (justify right bottom))
   )
-  (label "~{BUSACK}" (at 101.6 160.274 180) (fields_autoplaced)
-    (effects (font (size 1.27 1.27)) (justify right bottom))
-  )
   (label "D6" (at 158.75 93.472 180) (fields_autoplaced)
     (effects (font (size 1.27 1.27)) (justify right bottom))
@@
     (effects (font (size 1.27 1.27)) (justify right bottom))
   )
+  (label "~{NMI}" (at 103.378 50.292 0) (fields_autoplaced)
+    (effects (font (size 1.27 1.27)) (justify left bottom))
+  )
   (label "D7" (at 158.75 96.012 180) (fields_autoplaced)

Commit message: .
Parts:
- removed C?: 1uF, symbol Device:C
- removed D3: LED, symbol Device:LED
- removed D?: 1N4148, Diode_THT:D_DO-35_SOD27_P7.62mm_Horizontal, symbol Diode:1N4148
- removed J2: Conn_01x22, symbol Connector_Generic:Conn_01x22
- removed J5: Ext. Clock, symbol Connector_Generic:Conn_01x04
- removed R1: 10k, symbol Device:R
- removed R8: 220, symbol Device:R
- removed R?: 1K, symbol Device:R_US
- removed R?: 100, symbol Device:R_US
- removed SW?: RESET, symbol Switch:SW_Push
- added C1, C2: 10uF, symbol Device:C
- added J11: IO3, symbol Connector_Generic:Conn_01x08
- added J12: Ext. Clock, symbol Connector_Generic:Conn_02x03_Counter_Clockwise
- added J2: IO2, symbol Connector_Generic:Conn_01x08
- added J7: IO1, symbol Connector_Generic:Conn_01x08
- added R6: 10k, symbol Device:R
Connections:
- net +5V: now also C1.1, C2.1, J12.1 (Pin_1), J7.1 (Pin_1), R6.1
- net A0: now also J1.26 (Pin_26), J7.2 (Pin_2); no longer J1.28 (Pin_28)
- net A1: now also J1.17 (Pin_17), J7.3 (Pin_3); no longer J1.29 (Pin_29)
- net A10: now also J4.31 (Pin_31); no longer J4.8 (Pin_8)
- net A11: now also J4.2 (Pin_2); no longer J4.6 (Pin_6)
- net A12: now also J4.30 (Pin_30); no longer J1.36 (Pin_36)
- net A14: now also J4.29 (Pin_29); no longer J1.7 (Pin_7)
- net A15: now also J4.4 (Pin_4); no longer J4.32 (Pin_32)
- net A16: now also J1.30 (Pin_30), J7.5 (Pin_5); no longer J1.8 (Pin_8)
- net A17: now also J1.31 (Pin_31), J7.6 (Pin_6); no longer J4.1 (Pin_1)
- net A18: now also J1.32 (Pin_32), J7.7 (Pin_7); no longer J1.9 (Pin_9)
- net A2: now also J1.25 (Pin_25), J7.4 (Pin_4); no longer J1.30 (Pin_30)
- net A3: now also J1.18 (Pin_18); no longer J1.31 (Pin_31)
- net A4: now also J1.24 (Pin_24); no longer J1.32 (Pin_32)
- net A5: now also J1.19 (Pin_19); no longer J1.33 (Pin_33)
- net A6: now also J1.23 (Pin_23); no longer J1.34 (Pin_34)
- net A7: now also J1.20 (Pin_20); no longer J1.35 (Pin_35)
- net A8: now also J4.32 (Pin_32); no longer J4.4 (Pin_4)
- net A9: now also J4.1 (Pin_1); no longer J4.5 (Pin_5)
- net D0: now also J4.28 (Pin_28), J2.1 (Pin_1); no longer J1.27 (Pin_27)
- net D1: now also J4.5 (Pin_5), J2.2 (Pin_2); no longer J1.26 (Pin_26)
- net D2: now also J4.27 (Pin_27), J2.3 (Pin_3); no longer J1.25 (Pin_25)
- net D3: now also J4.6 (Pin_6), J2.4 (Pin_4); no longer J4.14 (Pin_14)
- net D4: now also J4.26 (Pin_26), J2.5 (Pin_5); no longer J4.13 (Pin_13)
- net D5: now also J4.7 (Pin_7), J2.6 (Pin_6); no longer J4.12 (Pin_12)
- net D6: now also J4.25 (Pin_25), J2.7 (Pin_7); no longer J4.11 (Pin_11)
- net D7: now also J4.8 (Pin_8), J2.8 (Pin_8); no longer J4.10 (Pin_10)
- net GND: now also C1.2, C2.2, J11.8 (Pin_8), J12.3 (Pin_3)
- net ~{BUSACK}: now also J4.18 (Pin_18); no longer J4.24 (Pin_24)
- net ~{BUSRQ}: now also J4.19 (Pin_19); no longer J4.25 (Pin_25)
- net ~{CLKENA}: now also J4.15 (Pin_15), SW2.1, J12.2 (Pin_2), R6.2; no longer J4.28 (Pin_28)
- net ~{CLK}: now also J4.16 (Pin_16), U2.6 (~{CLK}), J12.6 (Pin_6); no longer J4.29 (Pin_29)
- net ~{IORQ}: now also J4.17 (Pin_17), J11.1 (Pin_1); no longer J4.26 (Pin_26)
- net ~{IO_CE}: now also J4.12 (Pin_12), J11.6 (Pin_6); no longer J4.31 (Pin_31)
- net ~{M1}: now also J4.22 (Pin_22); no longer J4.27 (Pin_27)
- net ~{MREQ}: now also J1.27 (Pin_27), J11.2 (Pin_2); no longer J4.9 (Pin_9)
- net ~{NMI}: now also J4.11 (Pin_11); no longer J4.23 (Pin_23)
- net ~{RD}: now also J1.28 (Pin_28); no longer J4.7 (Pin_7)
- net ~{RST}: now also J4.21 (Pin_21), J11.5 (Pin_5); no longer J4.30 (Pin_30)
- net ~{WAIT}: now also J4.20 (Pin_20), J11.4 (Pin_4); no longer J4.22 (Pin_22)
- net ~{WR}: now also J1.29 (Pin_29), J11.3 (Pin_3); no longer J4.2 (Pin_2)
- no-connect marks 3 -> 40
Other:
- note added: "CLOCK"
- note added: "PA"
- note added: "PB4"
- note added: "PB6"
- note added: "PC0"
- note added: "PC1"
- note added: "PD1"
- note added: "PD3"
- note added: "PD7"
- note added: "PF"
- note added: "PG1"
- note added: "PG2"
- note added: "PH1"
- note added: "PJ1"
- note added: "PK"
- note added: "PL2"
- note added: "PL3"
- note added: "PL4"
- note added: "PL5"
- note added: "PL7"
- note removed: "RESET"
- moved on the sheet: J4
