File: circuit/io.kicad_sch (KiCad schematic)
At the start: 16 parts, among them J1 Micro_SD_Card, J2 VGA, J7 IO, J9 SWD programmer, SW1 Reset, U1 Pico, U10 TXB0104D, U4 TXS0108EPW, U7 74LS393

Commit message: .
Parts:
- removed J7: IO, symbol Connector_Generic:Conn_01x21
- added J2: Conn_01x22, symbol Connector_Generic:Conn_01x22
Connections:
- net +5V: now also J2.1 (Pin_1)
- net 5V_A0: now also J2.2 (Pin_2)
- net 5V_A1: now also J2.3 (Pin_3)
- net 5V_A16: now also J2.17 (Pin_17)
- net 5V_A17: now also J2.18 (Pin_18)
- net 5V_A18: now also J2.19 (Pin_19)
- net 5V_A2: now also J2.4 (Pin_4)
- net 5V_D0: now also J2.5 (Pin_5)
- net 5V_D1: now also J2.6 (Pin_6)
- net 5V_D2: now also J2.7 (Pin_7)
- net 5V_D3: now also J2.8 (Pin_8)
- net 5V_D4: now also J2.9 (Pin_9)
- net 5V_D5: now also J2.10 (Pin_10)
- net 5V_D6: now also J2.11 (Pin_11)
- net 5V_D7: now also J2.12 (Pin_12)
- net GND: now also J2.21 (Pin_21), J2.22 (Pin_22)
- net ~{5V_IORQ}: now also J2.13 (Pin_13)
- net ~{5V_MREQ}: now also J2.14 (Pin_14)
- net ~{5V_RST}: now also J2.20 (Pin_20)
- net ~{5V_WAIT}: now also J2.16 (Pin_16)
- net ~{5V_WR}: now also J2.15 (Pin_15)
Other:
- note added: "BANKSWITCHING"
- note added: "CONTROLLER"
- note added: "LEVEL SHIFTING (5v to 3v3)"
- note added: "STORAGE"
- note added: "VGA"
- moved on the sheet: U7A

Commit message: .
Parts:
- removed J2: Conn_01x22, symbol Connector_Generic:Conn_01x22
- removed U10: TXB0104D, Package_SO:SOIC-14_3.9x8.7mm_P1.27mm, symbol Logic_LevelTranslator:TXB0104D
- added J11: IO3, symbol Connector_Generic:Conn_01x08
- added J2: IO2, symbol Connector_Generic:Conn_01x08
- added J7: IO1, symbol Connector_Generic:Conn_01x08
- added U4: TXS0108EPW, Package_SO:TSSOP-20_4.4x6.5mm_P0.65mm, symbol Logic_LevelTranslator:TXS0108EPW
Connections:
- net +3V3: now also U4.10 (OE), U4.10 (OE), U4.2 (VCCA), U4.2 (VCCA), U4.10 (OE), U4.2 (VCCA); no longer U4.19 (VCCB), U4.19 (VCCB)
- net +5V: now also U4.19 (VCCB), U4.19 (VCCB), J7.1 (Pin_1), U4.19 (VCCB); no longer U4.2 (VCCA), U4.2 (VCCA)
- net 5V_A0: now also U4.20 (B1), J7.2 (Pin_2); no longer U4.1 (A1)
- net 5V_A1: now also U4.18 (B2), J7.3 (Pin_3); no longer U4.3 (A2)
- net 5V_A16: now also U4.16 (B4), J7.5 (Pin_5)
- net 5V_A17: now also U4.15 (B5), J7.6 (Pin_6)
- net 5V_A18: now also U4.14 (B6), J7.7 (Pin_7)
- net 5V_A2: now also U4.17 (B3), J7.4 (Pin_4); no longer U4.4 (A3)
- net 5V_D0: now also U4.20 (B1), J2.1 (Pin_1); no longer U4.5 (A4)
- net 5V_D1: now also U4.18 (B2), J2.2 (Pin_2); no longer U4.6 (A5)
- net 5V_D2: now also U4.17 (B3), J2.3 (Pin_3); no longer U4.7 (A6)
- net 5V_D3: now also U4.16 (B4), J2.4 (Pin_4); no longer U4.8 (A7)
- net 5V_D4: now also U4.15 (B5), J2.5 (Pin_5); no longer U4.9 (A8)
- net 5V_D5: now also U4.14 (B6), J2.6 (Pin_6); no longer U4.1 (A1)
- net 5V_D6: now also U4.13 (B7), J2.7 (Pin_7); no longer U4.3 (A2)
- net 5V_D7: now also U4.12 (B8), J2.8 (Pin_8); no longer U4.4 (A3)
- net A0: now also U4.1 (A1); no longer U4.20 (B1)
- net A1: now also U4.3 (A2); no longer U4.18 (B2)
- net A16: now also U4.5 (A4)
- net A17: now also U4.6 (A5)
- net A18: now also U4.7 (A6)
- net A2: now also U4.4 (A3); no longer U4.17 (B3)
- net D0: now also U4.1 (A1); no longer U4.16 (B4)
- net D1: now also U4.3 (A2); no longer U4.15 (B5)
- net D2: now also U4.4 (A3); no longer U4.14 (B6)
- net D3: now also U4.5 (A4); no longer U4.13 (B7)
- net D4: now also U4.6 (A5); no longer U4.12 (B8)
- net D5: now also U4.7 (A6); no longer U4.20 (B1)
- net D6: now also U4.8 (A7); no longer U4.18 (B2)
- net D7: now also U4.9 (A8); no longer U4.17 (B3)
- net GND: now also J11.8 (Pin_8), U4.11 (GND); no longer U4.10 (OE), U4.10 (OE)
- net ~{5V_IORQ}: now also J11.1 (Pin_1), U4.20 (B1); no longer U4.5 (A4)
- net ~{5V_MREQ}: now also J11.2 (Pin_2), U4.18 (B2); no longer U4.6 (A5)
- net ~{5V_RST}: now also J11.5 (Pin_5), U4.15 (B5)
- net ~{5V_WAIT}: now also J11.4 (Pin_4), U4.16 (B4); no longer U4.8 (A7)
- net ~{5V_WR}: now also J11.3 (Pin_3), U4.17 (B3); no longer U4.7 (A6)
- net ~{IORQ}: now also U4.1 (A1); no longer U4.16 (B4)
- net ~{MREQ}: now also U4.3 (A2); no longer U4.15 (B5)
- net ~{RST}: now also U4.6 (A5)
- net ~{WAIT}: now also U4.5 (A4); no longer U4.13 (B7)
- net ~{WR}: now also U4.4 (A3); no longer U4.14 (B6)
- new net ~{5V_IO_CE}: J11.6 (Pin_6), U4.14 (B6)
- new net ~{IO_CE}: U4.7 (A6)
- no-connect marks 25 -> 33

Commit message: .
Parts:
- removed J11: IO3, symbol Connector_Generic:Conn_01x08
- removed J2: IO2, symbol Connector_Generic:Conn_01x08
- removed J7: IO1, symbol Connector_Generic:Conn_01x08
- removed U4: TXS0108EPW, Package_SO:TSSOP-20_4.4x6.5mm_P0.65mm, symbol Logic_LevelTranslator:TXS0108EPW
- added J13: IO3, symbol Connector_Generic:Conn_01x08
- added J3: IO1, symbol Connector_Generic:Conn_01x08
- added J5: IO2, symbol Connector_Generic:Conn_01x08
- added U2: TXB0104RGY, Package_DFN_QFN:Texas_S-PVQFN-N14, symbol Logic_LevelTranslator:TXB0104RGY
- renumbered J2 to J10, J1 to J6, U7 to U11, U1 to U12, U4 to U14, U4 to U15
Connections:
- net +5V: now also J3.1 (Pin_1)
- net 5V_A0: now also J3.2 (Pin_2)
- net 5V_A1: now also J3.3 (Pin_3)
- net 5V_A16: now also J3.5 (Pin_5)
- net 5V_A17: now also J3.6 (Pin_6)
- net 5V_A18: now also J3.7 (Pin_7)
- net 5V_D0: now also J5.1 (Pin_1)
- net 5V_D1: now also J5.2 (Pin_2)
- net 5V_D2: now also J5.3 (Pin_3)
- net 5V_D3: now also J5.4 (Pin_4)
- net 5V_D4: now also J5.5 (Pin_5)
- net 5V_D5: now also J5.6 (Pin_6)
- net 5V_D6: now also J5.7 (Pin_7)
- net 5V_D7: now also J5.8 (Pin_8)
- net A2: no longer U14.4 (A3)
- net GND: now also U11.12 (MR), U11.13 (CP), J13.6 (Pin_6), J13.8 (Pin_8); no longer U11.1 (CP), U11.2 (MR)
- net ~{IORQ}: now also J13.1 (Pin_1), U2.13 (B1), U2.2 (A1)
- net ~{WAIT}: now also J13.4 (Pin_4), U2.11 (B3), U2.4 (A3)
- net ~{WR}: now also J13.3 (Pin_3), U2.12 (B2), U2.3 (A2)
- net 5V_A2: no longer names the net of U14.17 (B3)
- no-connect marks 33 -> 31
Other:
- note added: "I/O"
- moved on the sheet: J10, R10, R11, R12, R13, R14, U14, U15

Commit message: .
Parts:
- removed U2: TXB0104RGY, Package_DFN_QFN:Texas_S-PVQFN-N14, symbol Logic_LevelTranslator:TXB0104RGY
Connections:
- net A2 is gone; now on net D7: U12.12 (GPIO9)
- net 5V_D0: now also U14.15 (B5); no longer U15.20 (B1)
- net 5V_D1: now also U14.14 (B6); no longer U15.18 (B2)
- net 5V_D2: now also U14.13 (B7); no longer U15.17 (B3)
- net 5V_D3: now also U14.12 (B8); no longer U15.16 (B4)
- net 5V_D4: now also U15.20 (B1); no longer U15.15 (B5)
- net 5V_D5: now also U15.18 (B2); no longer U15.14 (B6)
- net 5V_D6: now also U15.17 (B3); no longer U15.13 (B7)
- net 5V_D7: now also U15.16 (B4); no longer U15.12 (B8)
- net A0: now also U12.1 (GPIO0); no longer U12.6 (GPIO4)
- net A1: now also U12.2 (GPIO1); no longer U12.10 (GPIO7)
- net A16: now also J3.5 (Pin_5); no longer U14.5 (A4)
- net A17: now also J3.6 (Pin_6); no longer U14.6 (A5)
- net A18: now also J3.7 (Pin_7); no longer U14.7 (A6)
- net BANK: now also U12.22 (GPIO17); no longer U12.9 (GPIO6)
- net BLUE: no longer U12.1 (GPIO0)
- net CSYNC: no longer U12.11 (GPIO8)
- net D0: now also U12.4 (GPIO2), U14.6 (A5); no longer U12.19 (GPIO14), U15.1 (A1)
- net D1: now also U12.5 (GPIO3), U14.7 (A6); no longer U12.20 (GPIO15), U15.3 (A2)
- net D2: now also U12.6 (GPIO4), U14.8 (A7); no longer U12.21 (GPIO16), U15.4 (A3)
- net D3: now also U12.7 (GPIO5), U14.9 (A8); no longer U12.22 (GPIO17), U15.5 (A4)
- net D4: now also U12.9 (GPIO6), U15.1 (A1); no longer U12.24 (GPIO18), U15.6 (A5)
- net D5: now also U12.10 (GPIO7), U15.3 (A2); no longer U12.25 (GPIO19), U15.7 (A6)
- net D6: now also U12.11 (GPIO8), U15.4 (A3); no longer U12.26 (GPIO20), U15.8 (A7)
- net D7: now also U15.5 (A4); no longer U12.27 (GPIO21), U15.9 (A8)
- net GREEN0: no longer U12.4 (GPIO2)
- net GREEN1: no longer U12.5 (GPIO3)
- net RED: no longer U12.7 (GPIO5)
- net ~{IORQ}: now also U12.19 (GPIO14), U15.8 (A7); no longer J13.1 (Pin_1), U12.2 (GPIO1)
- net ~{RST}: now also J13.7 (Pin_7); no longer U12.31 (GPIO26_ADC0)
- net ~{WAIT}: now also U12.21 (GPIO16); no longer U12.29 (GPIO22)
- net ~{WR}: now also U12.20 (GPIO15), U15.9 (A8); no longer J13.3 (Pin_3), U12.32 (GPIO27_ADC1)
- net 5V_A16: no longer names the net of U14.16 (B4)
- net 5V_A16: no longer J3.5 (Pin_5)
- removed net 5V_A17: J3.6 (Pin_6), U14.15 (B5)
- removed net 5V_A18: J3.7 (Pin_7), U14.14 (B6)
- net ~{MREQ}: no longer names the net of U12.34 (GPIO28_ADC2)
- new net ~{5V_IORQ}: J13.1 (Pin_1), U15.13 (B7)
- new net ~{5V_WR}: J13.3 (Pin_3), U15.12 (B8)
- no-connect marks 31 -> 35
Other:
- note added: "(connect to 5V)"
- moved on the sheet: J13, J5, U11B

Commit message: .
Parts:
- removed SW1: Reset, symbol Switch:SW_Push
- added U2: 74HC04, symbol 74xx:74HC04
Connections:
- net CSYNC: now also U12.32 (GPIO27_ADC1)
- net GREEN0: now also U12.27 (GPIO21)
- net GREEN1: now also U12.26 (GPIO20)
- net ~{IORQ}: now also U12.20 (GPIO15); no longer U12.19 (GPIO14)
- net ~{RST}: now also U12.30 (RUN), U15.7 (A6); no longer J13.7 (Pin_7)
- net ~{WR}: now also U12.19 (GPIO14); no longer U12.20 (GPIO15)
- net ~{5V_RST}: now reaches U15.14 (B6)
- net ~{5V_RST}: now also J13.5 (Pin_5), U2.1
- net BLUE0: now reaches U12.24 (GPIO18)
- net BLUE1: now reaches U12.25 (GPIO19)
- net RED0: now reaches U12.29 (GPIO22)
- net RED1: now reaches U12.31 (GPIO26_ADC0)
- net RST: no longer names the net of U11.2 (MR)
- net RST: now also U2.2
- no-connect marks 35 -> 33
Other:
- moved on the sheet: J10, R10, R11, R12, R13, R14
